Commit message: changes to camera height

File: CMP9767M/uol_cmp9767m_base/urdf/sensors.xacro (robot description, xacro)
@@ -256,5 +256,5 @@
         <mesh filename="package://kinect2_description/meshes/sensors/kinect2.dae"/>
       </geometry>
-      <origin xyz="0.02 0 0" rpy="0 0 3.141592"/>
+      <origin xyz="0.02 10 0" rpy="0 0 3.141592"/>
     </visual>
     <collision>
