Commit message: 1.) I've added the second robot - called robot_explorer - to the thorvald-sim.launch files and created a seperate launcher for it - that way we can edit our explorer robot with out changing the other robot. 2.) I've added a second xacro file (in the urdf folder) for the explorer robot to add to the camera's height etc. if you want to increase or decrease just edit line 266 :D 3.) I've set up another package for the MV and control code for the explorer robot called thorvald_explorer.

File: CMP9767M/uol_cmp9767m_base/urdf/sensors_explorer.xacro (robot description, xacro)
@@ -247,5 +247,5 @@
   <xacro:property name="kinect2_cam_px" value="0.45" />
   <xacro:property name="kinect2_cam_py" value="0.0" />
-  <xacro:property name="kinect2_cam_pz" value="0.5" />
+  <xacro:property name="kinect2_cam_pz" value="20.5" />
   <xacro:property name="kinect2_cam_or" value="0.0" />
   <xacro:property name="kinect2_cam_op" value="${M_PI/2}" />
@@ -300,5 +300,5 @@
         <clip>
           <near>0.1</near>
-          <far>8.0</far>
+          <far>100.0</far>
         </clip>
         <noise>
@@ -322,5 +322,5 @@
         <frameName>${kinect2_name}_depth_optical_frame</frameName>
         <pointCloudCutoff>0.5</pointCloudCutoff>
-        <pointCloudCutoffMax>8.0</pointCloudCutoffMax>
+        <pointCloudCutoffMax>100.0</pointCloudCutoffMax>
         <baseline>0.1</baseline>
         <distortionK1>0.0</distortionK1>
@@ -346,5 +346,5 @@
         <clip>
           <near>0.02</near>
-          <far>10.0</far>
+          <far>100.0</far>
         </clip>
         <noise>

Commit message: I moved the explorer robot out of the way while the camera stays in the middle of the field. Couldn't figure out how to make the model invisible.

File: CMP9767M/uol_cmp9767m_base/urdf/sensors_explorer.xacro (robot description, xacro)
@@ -245,6 +245,6 @@
   <xacro:property name="kinect2_parent" value="base_link" />
   <xacro:property name="kinect2_name" value="kinect2" />
-  <xacro:property name="kinect2_cam_px" value="0.45" />
-  <xacro:property name="kinect2_cam_py" value="0.0" />
+  <xacro:property name="kinect2_cam_px" value="10.0" />
+  <xacro:property name="kinect2_cam_py" value="10.0" />
   <xacro:property name="kinect2_cam_pz" value="20.5" />
   <xacro:property name="kinect2_cam_or" value="0.0" />
